Commit message: Changed path to mesh

File: Laba_2/urdf/car.xacro (robot description, xacro)
@@ -71,5 +71,5 @@
       <origin xyz="0 0 0" rpy="0 0 0"/>
       <geometry>
-        <mesh filename="/home/master/Desktop/II_last_semester/Laba_2/meshes/car.dae"/>
+        <mesh filename="../meshes/car.dae"/>
       </geometry>
     </visual>
@@ -193,5 +193,5 @@
       <origin xyz="0 0 0" rpy="0 0 0"/>
       <geometry>
-        <mesh filename="/home/master/Desktop/II_last_semester/Laba_2/meshes/hokuyo.dae"/>
+        <mesh filename="../meshes/hokuyo.dae"/>
       </geometry>
     </visual>

File: Laba_2/urdf/map.xacro (robot description, xacro)
@@ -5,5 +5,5 @@
       <origin xyz="0 0 0" rpy="0 0 0"/>
       <geometry>
-        <mesh filename="../meshes/map.dae"/>
+        <mesh filename="package://ackermann_vehicle_description/meshes/map.dae"/>
       </geometry>
     </collision>
@@ -11,5 +11,5 @@
       <origin xyz="0 0 0" rpy="0 0 0"/>
       <geometry>
-        <mesh filename="../meshes/map.dae"/>
+        <mesh filename="package://ackermann_vehicle_description/meshes/map.dae"/>
       </geometry>
     </visual>
